Commit message: added rviz rendering with moveit support as a launch argument from description

File: src/description/urdf/robot_cell_macro.xacro (robot description, xacro)
@@ -2,5 +2,5 @@
 <robot xmlns:xacro="http://ros.org/wiki/xacro">
     <xacro:include filename="$(find ur_description)/urdf/ur_macro.xacro"/>
-    <xacro:macro name="my_robot_cell" params="
+    <xacro:macro name="robot_cell" params="
     parent
     *origin
@@ -11,77 +11,13 @@
     visual_parameters_file
     ">
-        <joint name="table_base_joint" type="fixed">
-            <xacro:insert_block name="origin" />
-            <parent link="${parent}" />
-            <child link="table" />
-        </joint>
-        <link name="table">
-            <visual>
-                <geometry>
-                    <mesh filename="package://my_robot_cell_description/meshes/fzi_table.dae"/>
-                </geometry>
-                <origin rpy="0 0 0" xyz="0.75 0.5 -1"/>
-            </visual>
-            <collision>
-                <geometry>
-                    <mesh filename="package://my_robot_cell_description/meshes/fzi_table.dae"/>
-                </geometry>
-                <origin rpy="0 0 0" xyz="0.75 0.5 -1"/>
-            </collision>
-        </link>
-        <link name="monitor">
-            <visual>
-                <geometry>
-                    <mesh filename="package://my_robot_cell_description/meshes/171005_Motek_Monitor_L.dae"/>
-                </geometry>
-            </visual>
-            <collision>
-                <geometry>
-                    <mesh filename="package://my_robot_cell_description/meshes/171005_Motek_Monitor_L.dae"/>
-                </geometry>
-            </collision>
-        </link>
-        <joint name="base_to_monitor" type="fixed">
-            <parent link="table"/>
-            <child link="monitor"/>
-            <origin xyz="0.2 0.6 0"/>
-        </joint>
-        <material name="white">
-            <color rgba="1 1 1 1"/>
-        </material>
-        <link name="wall">
-            <visual>
-                <geometry>
-                    <mesh filename="package://my_robot_cell_description/meshes/wall.dae"/>
-                </geometry>
-            </visual>
-            <collision>
-                <geometry>
-                    <box size="4.44 0.1 2.5"/>
-                </geometry>
-            </collision>
-        </link>
-        <joint name="base_to_wall" type="fixed">
-            <parent link="table"/>
-            <child link="wall"/>
-            <origin xyz="1.25 1.5 0.5"/>
-        </joint>
-        <link name="robot_mount"/>
-        <joint name="base_to_robot_mount" type="fixed">
-            <parent link="table"/>
-            <child link="robot_mount"/>
-            <origin xyz="0.845 0.85 0" rpy="0 0 ${pi}" />
-        </joint>
-        <!--This will create the specific robot-->
         <xacro:ur_robot
-                name="${ur_type}"
-                tf_prefix="${ur_type}_"
-                parent="robot_mount"
-                joint_limits_parameters_file="${joint_limits_parameters_file}"
-                kinematics_parameters_file="${kinematics_parameters_file}"
-                physical_parameters_file="${physical_parameters_file}"
-                visual_parameters_file="${visual_parameters_file}"
-        >
-            <origin xyz="0 0 0" rpy="0 0 0" />
+            name="${ur_type}"
+            tf_prefix="${ur_type}_"
+            parent="${parent}"
+            joint_limits_parameters_file="${joint_limits_parameters_file}"
+            kinematics_parameters_file="${kinematics_parameters_file}"
+            physical_parameters_file="${physical_parameters_file}"
+            visual_parameters_file="${visual_parameters_file}">
+            <xacro:insert_block name="origin"/>
         </xacro:ur_robot>
     </xacro:macro>

Commit message: Big commit but most is from ur moveit tutorials

File: src/description/urdf/robot_cell_macro.xacro (robot description, xacro)
@@ -2,4 +2,5 @@
 <robot xmlns:xacro="http://ros.org/wiki/xacro">
     <xacro:include filename="$(find ur_description)/urdf/ur_macro.xacro"/>
+    <xacro:include filename="$(find description)/urdf/gripper_macro.xacro"/>
     <xacro:macro name="robot_cell" params="
     parent
@@ -11,14 +12,63 @@
     visual_parameters_file
     ">
+        <joint name="base_plate" type="fixed">
+            <xacro:insert_block name="origin"/>
+            <parent link="${parent}"/>
+            <child link="base_plate"/>
+        </joint>
+        <link name="base_plate">
+            <visual>
+                <geometry>
+                    <mesh filename="package://description/meshes/table/BasePlate.stl" scale="0.001 0.001 0.001"/>
+                </geometry>
+                <origin xyz="0 0 0" rpy="${pi/2} 0 ${pi/2}" />
+                <material name="aluminum">
+                    <color rgba="0.77 0.78 0.80 1.0"/>
+                </material>
+            </visual>
+            <collision>
+                <geometry>
+                    <mesh filename="package://description/meshes/table/BasePlate.stl" scale="0.001 0.001 0.001"/>
+                </geometry>
+                <origin xyz="0 0 0" rpy="${pi/2} 0 ${pi/2}" />
+            </collision>
+        </link>
+        <link name="Eevee_base_plate">
+            <visual>
+                <geometry>
+                    <mesh filename="package://description/meshes/table/EeveeMountingPlate.stl" scale="0.001 0.001 0.001"/>
+                </geometry>
+                <origin xyz="0 0 0" rpy="0 0 ${pi/2}" />
+                <material name="aluminum">
+                    <color rgba="0.77 0.78 0.80 1.0"/>
+                </material>
+            </visual>
+            <collision>
+                <geometry>
+                    <mesh filename="package://description/meshes/table/EeveeMountingPlate.stl" scale="0.001 0.001 0.001"/>
+                </geometry>
+                <origin xyz="0 0 0" rpy="0 0 ${pi/2}" />
+            </collision>
+        </link>
+        <joint name="base_plate_to_Eevee_base_plate" type="fixed">
+            <parent link="base_plate"/>
+            <child link="Eevee_base_plate"/>
+            <origin xyz="0 0.5 0" rpy="0 0 0" />
+        </joint>
         <xacro:ur_robot
             name="${ur_type}"
             tf_prefix="${ur_type}_"
-            parent="${parent}"
+            parent="Eevee_base_plate"
             joint_limits_parameters_file="${joint_limits_parameters_file}"
             kinematics_parameters_file="${kinematics_parameters_file}"
             physical_parameters_file="${physical_parameters_file}"
             visual_parameters_file="${visual_parameters_file}">
-            <xacro:insert_block name="origin"/>
+            <origin xyz="0 0 0.01" rpy="0 0 0"/>
         </xacro:ur_robot>
+        <xacro:gripper
+                parent="${ur_type}_tool0"
+                prefix="${ur_type}_">
+            <origin xyz="0 0 0" rpy="0 0 0"/>
+        </xacro:gripper>
     </xacro:macro>
 </robot>
